Commit message: feat: d405 capture 적용

File: robot/urdf/omx_f/omx_f.urdf (robot description, URDF)
Before this commit: robot omx_f, 10 links, 9 joints
Links:
- link link5: geometry collision mesh filename=../../meshes/omx_f/follower_06_pan_Revised_d405.stl scale=0.001 0.001 0.001; visual mesh filename=../../meshes/omx_f/follower_06_pan_Revised_d405.stl scale=0.001 0.001 0.001
