Commit message: refactor: robot/ → type/instance split + RobotRegistry (multi_robot §4/§5)
multi_robot_architecture.md §4 (Robot identity) / §5 (디렉토리 구조) 의 LeRobot 식
type/instance split 적용. Phase 1 single robot (omx_f_0) 만 있는 상태에서 그대로
SO-101 plug-and-play 가능한 abstraction 깔기.

폴더 구조:
- robot/urdf/omx_f/{omx_f.urdf,meshes/} → robot/omx_f/urdf/{omx_f.urdf,meshes/}
  (type 폴더, URDF mesh path 도 `meshes/` 상대경로로 갱신)
- robot/calibration/*.npz (7종) → robot/instances/omx_f_0/calibration/
- robot/config/motors.yaml split:
  · type-level (motors 리스트, joint limit, gear ratio, PID) → robot/omx_f/motors.yaml
  · instance-level (port, baudrate) → robot/instances/omx_f_0/instance.yaml
- robot/config/robot_poses.yaml → robot/instances/omx_f_0/robot_poses.yaml
- robot/models/, robot/scans/, robot/logs/ → robot/instances/omx_f_0/{meshes/,scans/,logs/}
- robot/robots.yaml (★ 신규) — top-level registry

코드:
- backend/core/robot_registry.py (★ 신규) — RobotRegistry 싱글톤. robots.yaml 1회
  load + per-robot RobotConfig 조립 (type/instance path 자동 계산). reserved name
  validation (system/task/coord/viz/cameras + instances/extrinsics/workspace 등
  robot_id 로 사용 금지). default() = N=1 편의 메서드.
- core/{joint,link,sag,tool}_coordinates.py — path 상수 → RobotRegistry().default().
  calibration_dir / *.npz 동적 lookup
- core/robot_poses.py — RobotRegistry path 사용
- modules/calibration/loader.py — CALIB_DIR → _calib_dir() 동적
- modules/dynamixel/motor_config.py — load_motor_config() 가 robot_id 인자 받아
  type motors.yaml + instance.yaml split load. legacy single-file loader 도 호환
  유지 (deprecated)
- modules/kinematics/solver.py — URDF_PATH 상수 제거, RobotRegistry().default().
  urdf_path 사용
- modules/pointcloud/scan_io.py — SCANS_DIR/MODELS_DIR/CALIB_DIR 상수 → 함수
  (_scans_dir / meshes_dir / _calib_dir / robot_root)
- nodes/calibration_node.py — SAVE_DIR / HANDEYE_POSES_PATH 함수화
- nodes/pointcloud_node.py — scan_io.MODELS_DIR → scan_io.meshes_dir(),
  scan_io.ROBOT_DIR → scan_io.robot_root()
- main.py — D405 intrinsic seed path 도 RobotRegistry

.gitignore:
- robot/urdf/**/.patched/ → robot/*/urdf/**/.patched/ (새 구조)
- robot/scans/ / robot/models/ → robot/instances/*/scans/ / robot/instances/*/meshes/
- robot/logs/ → robot/instances/*/logs/

검증:
- RobotRegistry load + 모든 calibration/urdf/config path 존재 확인
- JointCoordinates / LinkCoordinates / SagCoordinates / ToolCoordinates 로드
- robot_poses.yaml 로드 (home/rest/search_1/2/3)
- load_motor_config() type+instance split 정상 load (6 motors, port COM6)
- PybulletSolver FK 정상 (URDF + 새 mesh path + sag/link_offset 모두 적용)
- main.py boot 시 패치된 URDF 새 경로 (robot/omx_f/urdf/.patched/omx_f.urdf) 생성
- ruff + pyright clean on 변경 파일들 (pre-existing motion_node.py 의 ruff/pyright
  에러는 손대지 않음)

후속:
- RobotRegistry 위에서 robot_id 차원 도입 (JointStateCache / Coordinates 의
  dict[robot_id] 화) — 별도 todo

Co-Authored-By: Claude Opus 4.7 (1M context) <noreply@anthropic.com>

File: robot/omx_f/urdf/omx_f.urdf (robot description, URDF)
Before this commit: robot omx_f, 10 links, 9 joints
Links:
- link link0: geometry collision mesh filename=meshes/follower_01_base.stl scale=0.001 0.001 0.001; visual mesh filename=meshes/follower_01_base.stl scale=0.001 0.001 0.001
- link link1: geometry collision mesh filename=meshes/follower_02_base_tilt_Revised.stl scale=0.001 0.001 0.001; visual mesh filename=meshes/follower_02_base_tilt_Revised.stl scale=0.001 0.001 0.001
- link link2: geometry collision mesh filename=meshes/follower_03_middle_verticle.stl scale=0.001 0.001 0.001; visual mesh filename=meshes/follower_03_middle_verticle.stl scale=0.001 0.001 0.001
- link link3: geometry collision mesh filename=meshes/follower_04_middle_horizontal.stl scale=0.001 0.001 0.001; visual mesh filename=meshes/follower_04_middle_horizontal.stl scale=0.001 0.001 0.001
- link link4: geometry collision mesh filename=meshes/follower_05_tip.stl scale=0.001 0.001 0.001; visual mesh filename=meshes/follower_05_tip.stl scale=0.001 0.001 0.001
- link link5: geometry collision mesh filename=meshes/follower_06_pan_Revised_d405.stl scale=0.001 0.001 0.001; visual mesh filename=meshes/follower_06_pan_Revised_d405.stl scale=0.001 0.001 0.001
- link link6: geometry collision mesh filename=meshes/follower_07_gripper_motorized.stl scale=0.001 0.001 0.001; visual mesh filename=meshes/follower_07_gripper_motorized.stl scale=0.001 0.001 0.001
- link link7: geometry collision mesh filename=meshes/follower_08_gripper_gear.stl scale=0.001 0.001 0.001; visual mesh filename=meshes/follower_08_gripper_gear.stl scale=0.001 0.001 0.001
