Commit message: feat: 멀티로봇 대응 하드코딩들 제거

File: robot/omx_f/urdf/omx_f.urdf (robot description, URDF)
Before this commit: robot omx_f, 10 links, 9 joints
Links:
- removed link end_effector_link
- added link tcp; visual box size=0.01 0.01 0.01
Joints:
- removed joint end_effector_joint
- added joint tcp_joint: type fixed, parent link5, child tcp, origin xyz=0.09193 -0.0016 0 rpy=0 0 0
