Commit message: feat: so101 test...

File: robot/so101_6dof/urdf/so101_6dof.urdf (robot description, URDF)
Before this commit: robot so101_6dof, 14 links, 13 joints
Joints:
- joint joint2: origin xyz=0.0306 0.0183 -0.0542 rpy=1.5708 1.5708 0 -> xyz=0.0306 0.0183 -0.0542 rpy=1.5708 3.14159 0
- joint joint3: origin xyz=0.11257 0.028 -0 rpy=0 -0 1.5708 -> xyz=0.11257 0.028 -0 rpy=0 0 3.14159

Commit message: fix: so101 urdf 수정중

File: robot/so101_6dof/urdf/so101_6dof.urdf (robot description, URDF)
Before this commit: robot so101_6dof, 14 links, 13 joints
Links:
- removed link camera
- removed link camera_body
- removed link camera_mount
- link gripper_fixed: geometry visual mesh filename=meshes/sts3215.stl; visual mesh filename=meshes/wrist_roll_d405_holder.stl
Joints:
- removed joint camera
- removed joint camera_frame
- removed joint camera_mount

Commit message: feat: 모터 수정

File: robot/so101_6dof/urdf/so101_6dof.urdf (robot description, URDF)
Before this commit: robot so101_6dof, 11 links, 10 joints
Joints:
- joint joint1: limit lower=-1.91986 upper=1.91986 effort=3.3 velocity=5 -> lower=-1.5708 upper=1.5708 effort=3.3 velocity=5
- joint joint2: limit lower=-1.74533 upper=1.74533 effort=3.3 velocity=5 -> lower=0 upper=2.0944 effort=3.3 velocity=5
- joint joint3: limit lower=-1.68948 upper=1.5708 effort=3.3 velocity=5 -> lower=-2.0944 upper=0 effort=3.3 velocity=5
- joint joint4: limit lower=-1.46608 upper=1.64061 effort=3.3 velocity=5 -> lower=-1.22173 upper=1.22173 effort=3.3 velocity=5
- joint joint5: limit lower=-1.54481 upper=1.52697 effort=3.3 velocity=5 -> lower=-1.51844 upper=1.51844 effort=3.3 velocity=5
- joint joint6: limit lower=-2.97071 upper=2.85869 effort=3.3 velocity=5 -> lower=0 upper=3.14159 effort=3.3 velocity=5

Commit message: fix: 실시간 포인트 클라우드 버그 수정

File: robot/so101_6dof/urdf/so101_6dof.urdf (robot description, URDF)
Before this commit: robot so101_6dof, 11 links, 10 joints
Joints:
- joint joint2: limit lower=0 upper=2.0944 effort=3.3 velocity=5 -> lower=-0.174533 upper=2.61799 effort=3.3 velocity=5
- joint joint3: limit lower=-2.0944 upper=0 effort=3.3 velocity=5 -> lower=-3.05433 upper=-0.0872665 effort=3.3 velocity=5
- joint joint4: limit lower=-1.22173 upper=1.22173 effort=3.3 velocity=5 -> lower=-1.51844 upper=1.51844 effort=3.3 velocity=5
- joint tcp_joint: origin xyz=0 0 0 rpy=0 0 0 -> xyz=0.04 0 0 rpy=0 0 0

Commit message: feat: self collision 추가

File: robot/so101_6dof/urdf/so101_6dof.urdf (robot description, URDF)
Before this commit: robot so101_6dof, 11 links, 10 joints
Links:
- link base: geometry collision mesh filename=meshes/base.stl; collision mesh filename=meshes/base_motor_holder.stl
- link base_rotation: geometry collision mesh filename=meshes/arm_motor_holder.stl; collision mesh filename=meshes/base_rotation.stl
- link gripper_fixed: geometry collision mesh filename=meshes/sts3215.stl; collision mesh filename=meshes/wrist_roll_d405_holder.stl
- link gripper_jaw: geometry collision mesh filename=meshes/gripper_jaw.stl; visual mesh filename=meshes/gripper_jaw.stl
- link under_arm: geometry collision mesh filename=meshes/sts3215.stl; collision mesh filename=meshes/under_arm.stl
- link upper_arm: geometry collision mesh filename=meshes/sts3215.stl; collision mesh filename=meshes/upper_arm.stl
- link wrist_yaw_back: geometry collision mesh filename=meshes/wrist_yaw_back.stl; visual mesh filename=meshes/wrist_yaw_back.stl
- link wrist_yaw_front: geometry collision mesh filename=meshes/sts3215.stl; collision mesh filename=meshes/sts3215.stl
