Commit message: feat: omx enable

File: robot_v2/omx_f/urdf/omx_f.urdf (robot description, URDF)
Before this commit: robot omx_f, 10 links, 9 joints
Links:
- link link5: geometry collision mesh filename=meshes/follower_06_pan_Revised.stl scale=0.001 0.001 0.001; visual mesh filename=meshes/follower_06_pan_Revised.stl scale=0.001 0.001 0.001
Joints:
- joint gripper_joint_1: limit lower=-6.283185307179586 upper=6.283185307179586 effort=1000 velocity=4.8 -> lower=-0.3805 upper=0.8469 effort=1000 velocity=4.8
- joint gripper_joint_2: limit lower=-6.283185307179586 upper=6.283185307179586 effort=1000 velocity=4.8 -> lower=-0.8469 upper=0.3805 effort=1000 velocity=4.8
- joint joint1: limit lower=-6.283185307179586 upper=6.283185307179586 effort=1000 velocity=4.8 -> lower=-3.14159 upper=3.14159 effort=1000 velocity=4.8
- joint joint2: limit lower=-6.283185307179586 upper=6.283185307179586 effort=1000 velocity=4.8 -> lower=-1.5708 upper=1.5708 effort=1000 velocity=4.8
- joint joint3: limit lower=-6.283185307179586 upper=6.283185307179586 effort=1000 velocity=4.8 -> lower=-1.5708 upper=1.5708 effort=1000 velocity=4.8
- joint joint4: limit lower=-6.283185307179586 upper=6.283185307179586 effort=1000 velocity=4.8 -> lower=-1.5708 upper=1.5708 effort=1000 velocity=4.8
- joint joint5: limit lower=-6.283185307179586 upper=6.283185307179586 effort=1000 velocity=4.8 -> lower=-3.14159 upper=3.14159 effort=1000 velocity=4.8
